Commit message: Added robot body visuals

File: description/robot.urdf.xacro (robot description, xacro)
@@ -13,5 +13,65 @@
         <color rgba ="0 0 0 1" />
     </material>
+    <!-- BASE LINK -->
     <link name="base_link">
     </link>
+    <!-- CHASSIS LINK -->
+    <joint name="chassis_joint" type="fixed">
+        <parent link="base_link"/>
+        <child link="chassis" />
+        <origin xyz="-0.1 0 0" />
+    </joint>
+    <link name="chassis">
+        <visual>
+            <origin xyz="0.15 0 0.075"/>
+            <geometry>
+                <box size="0.3 0.3 0.15" />
+            </geometry>
+            <material name="white"/>
+        </visual>
+    </link>
+    <!-- LEFT WHEEL LINK -->
+    <joint name="left_wheel_joint" type="continuous">
+        <parent link="base_link" />
+        <child link="left_wheel" />
+        <origin xyz="0 0.175 0" rpy="-${pi/2} 0 0" />
+        <axis xyz="0 0 1" />
+    </joint>
+    <link name="left_wheel">
+        <visual>
+            <geometry>
+                <cylinder radius="0.05" length="0.04" />
+            </geometry>
+            <material name="blue" />
+        </visual>
+    </link>
+    <!-- RIGHT WHEEL LINK -->
+    <joint name="right_wheel_joint" type="continuous">
+        <parent link="base_link" />
+        <child link="right_wheel" />
+        <origin xyz="0 -0.175 0" rpy="+${pi/2} 0 0" />
+        <axis xyz="0 0 -1" />
+    </joint>
+    <link name="right_wheel">
+        <visual>
+            <geometry>
+                <cylinder radius="0.05" length="0.04" />
+            </geometry>
+            <material name="blue" />
+        </visual>
+    </link>
+    <!-- CASTER WHEEL LINK -->
+    <joint name="caster_wheel_joint" type="fixed">
+        <parent link="chassis" />
+        <child link="caster_wheel" />
+        <origin xyz="0.24 0 0" />
+    </joint>
+    <link name="caster_wheel">
+        <visual>
+            <geometry>
+                <sphere radius="0.05" />
+            </geometry>
+            <material name="black" />
+        </visual>
+    </link>
 </robot>

Commit message: Added robot body collision

File: description/robot.urdf.xacro (robot description, xacro)
@@ -30,4 +30,11 @@
             <material name="white"/>
         </visual>
+        <collision>
+            <origin xyz="0.15 0 0.075"/>
+            <geometry>
+                <box size="0.3 0.3 0.15" />
+            </geometry>
+            <material name="white"/>
+        </collision>
     </link>
     <!-- LEFT WHEEL LINK -->
@@ -45,4 +52,10 @@
             <material name="blue" />
         </visual>
+        <collsion>
+            <geometry>
+                <cylinder radius="0.05" length="0.04" />
+            </geometry>
+            <material name="blue" />
+        </collsion>
     </link>
     <!-- RIGHT WHEEL LINK -->
@@ -60,4 +73,10 @@
             <material name="blue" />
         </visual>
+        <collision>
+            <geometry>
+                <cylinder radius="0.05" length="0.04" />
+            </geometry>
+            <material name="blue" />
+        </collision>
     </link>
     <!-- CASTER WHEEL LINK -->
@@ -74,4 +93,10 @@
             <material name="black" />
         </visual>
+        <collision>
+            <geometry>
+                <sphere radius="0.05" />
+            </geometry>
+            <material name="black" />
+        </collision>
     </link>
 </robot>

Commit message: Added robot body inertias

File: description/robot.urdf.xacro (robot description, xacro)
@@ -1,4 +1,5 @@
 <?xml version="1.0"?>
 <robot xmlns:xacro="http://www.ros.org/wiki/xacro"  name="robot">
+    <xacro:include filename="inertial_macros.xacro" />
     <material name="white">
         <color rgba ="1 1 1 1" />
@@ -37,4 +38,7 @@
             <material name="white"/>
         </collision>
+        <xacro:inertial_box mass="0.5" x="0.3" y="0.3" z="0.15">
+            <origin xyz="0.15 0 0.075" rpy="0 0 0" />
+        </xacro:inertial_box>
     </link>
     <!-- LEFT WHEEL LINK -->
@@ -58,4 +62,7 @@
             <material name="blue" />
         </collsion>
+        <xacro:inertial_cylinder mass="0.1" length="0.04" radius="0.05">
+            <origin xyz="0 0 0" rpy="0 0 0"/>
+        </xacro:inertial_cylinder>
     </link>
     <!-- RIGHT WHEEL LINK -->
@@ -79,4 +86,7 @@
             <material name="blue" />
         </collision>
+        <xacro:inertial_cylinder mass="0.1" length="0.04" radius="0.05">
+            <origin xyz="0 0 0" rpy="0 0 0"/>
+        </xacro:inertial_cylinder>
     </link>
     <!-- CASTER WHEEL LINK -->
@@ -99,4 +109,7 @@
             <material name="black" />
         </collision>
+        <xacro:inertial_sphere mass="0.1" radius="0.05">
+            <origin xyz="0 0 0" rpy="0 0 0"/>
+        </xacro:inertial_sphere>
     </link>
 </robot>
