Commit message: Added depth camera - not working atm

File: description/rgb_camera.xacro (robot description, xacro)
@@ -1,10 +1,10 @@
 <?xml version="1.0"?>
 <robot xmlns:xacro="http://www.ros.org/wiki/xacro">
-    <joint name="camera_joint" type="fixed">
+    <joint name="rgb_camera_joint" type="fixed">
         <parent link="chassis" />
-        <child link="camera_link" />
+        <child link="rgb_camera_link" />
         <origin xyz="0.276 0.0 0.181" rpy="0.0 0.18 0.0" />
     </joint>
-    <link name="camera_link">
+    <link name="rgb_camera_link">
         <visual>
             <geometry>
@@ -21,11 +21,11 @@
         </visual>
     </link>
-    <joint name="camera_optical_joint" type="fixed">
-        <parent link="camera_link" />
-        <child link="camera_link_optical" />
+    <joint name="rgb_camera_optical_joint" type="fixed">
+        <parent link="rgb_camera_link" />
+        <child link="rgb_camera_link_optical" />
         <origin xyz="0.0 0.0 0.0" rpy="${-pi/2} 0 ${-pi/2}" />
     </joint>
-    <link name="camera_link_optical"> </link>
-    <gazebo reference="camera_link">
+    <link name="rgb_camera_link_optical"> </link>
+    <gazebo reference="rgb_camera_link">
         <sensor name="camera" type="camera">
             <pose> 0 0 0 0 0 0 </pose>
@@ -46,5 +46,5 @@
             </camera>
             <topic>camera/image_raw</topic>
-            <gz_frame_id>camera_link_optical</gz_frame_id>
+            <gz_frame_id>rgb_camera_link_optical</gz_frame_id>
         </sensor>
     </gazebo>

File: description/robot.urdf.xacro (robot description, xacro)
@@ -4,5 +4,6 @@
     <xacro:include filename="gazebo_control.xacro"/>
     <xacro:include filename="lidar.xacro"/>
-    <xacro:include filename="camera.xacro"/>
+    <xacro:include filename="rgb_camera.xacro"/>
+    <xacro:include filename="depth_camera.xacro"/>
     <!-- <xacro:include filename="ros2_control.xacro" /> -->
     <!-- <xacro:add_ros2_control left_joint="left_wheel_joint" right_joint="right_wheel_joint"/> -->
