Commit message: Working 2D slam with slam_toolbox

File: description/lidar.xacro (robot description, xacro)
@@ -1,4 +1,7 @@
 <?xml version="1.0"?>
 <robot xmlns:xacro="http://www.ros.org/wiki/xacro">
+    <material name="red">
+        <color rgba="1.0 0.0 0.0 1.0" />
+    </material>
     <joint name="laser_joint" type="fixed">
         <parent link="chassis" />
@@ -38,5 +41,10 @@
                     <min>0.3</min>
                     <max>12</max>
+                    <resolution>0.001</resolution>
                 </range>
+                <noise type="gaussian">
+                    <mean>0.0</mean>
+                    <stddev>0.01</stddev> <!-- 1 cm standard deviation -->
+                </noise>
             </lidar>
             <topic>scan</topic>
@@ -44,5 +52,5 @@
         </sensor>
     </gazebo>
-    <plugin name="laser_controller" filename="libgazebo_ros_ray_sensor.so">
+    <!-- <plugin name="laser_controller" filename="libgazebo_ros_ray_sensor.so">
         <ros>
             <argument>~/out:=scan</argument>
@@ -50,4 +58,4 @@
         <output_type>sensor_msgs/LaserScan</output_type>
         <frame_name>laser_frame</frame_name>
-    </plugin>
+    </plugin> -->
 </robot>

File: description/rgb_camera.xacro (robot description, xacro)
@@ -42,5 +42,5 @@
                 <clip>
                     <near>0.05</near>
-                    <far>8.0</far>
+                    <far>120.0</far>
                 </clip>
             </camera>

File: description/robot.urdf.xacro (robot description, xacro)
@@ -5,5 +5,5 @@
     <xacro:include filename="lidar.xacro"/>
     <xacro:include filename="rgb_camera.xacro"/>
-    <xacro:include filename="depth_camera.xacro"/>
+    <!-- <xacro:include filename="depth_camera.xacro"/> -->
     <!-- <xacro:include filename="ros2_control.xacro" /> -->
     <!-- <xacro:add_ros2_control left_joint="left_wheel_joint" right_joint="right_wheel_joint"/> -->
