Commit message: feat(localization): add robot_localization EKF sensor fusion with backend-aware TF ownership

File: description/gazebo_control.xacro (robot description, xacro)
@@ -1,29 +1,31 @@
 <?xml version="1.0"?>
 <robot xmlns:xacro="http://www.ros.org/wiki/xacro" name="robot">
-    <gazebo>
-        <plugin name='gz::sim::systems::DiffDrive' filename='gz-sim-diff-drive-system'>
-            <!-- WHEEL INFORMATION -->
-            <left_joint>left_wheel_joint</left_joint>
-            <right_joint>right_wheel_joint</right_joint>
-            <wheel_separation>0.35</wheel_separation>
-            <wheel_radius>0.05</wheel_radius>
-            <!-- LIMITS -->
-            <!-- <max_wheel_torque>200</max_wheel_torque> -->
-            <!-- <max_wheel_acceleration>10.0</max_wheel_acceleration> -->
-            <!-- INPUT -->
-            <topic>cmd_vel</topic>
-            <!-- OUTPUT -->
-            <frame_id>odom</frame_id>
-            <child_frame_id>base_link</child_frame_id>
-            <odom_topic>odom</odom_topic>
-            <tf_topic>/tf</tf_topic>
-            <!-- <odom_publisher_frequency>30</odom_publisher_frequency> -->
-        </plugin>
-        <plugin name="gz::sim::systems::JointStatePublisher"
-            filename="gz-sim-joint-state-publisher-system">
-            <topic>joint_states</topic>
-            <joint_name>left_wheel_joint</joint_name>
-            <joint_name>right_wheel_joint</joint_name>
-        </plugin>
-    </gazebo>
+    <xacro:unless value="${use_ros2_control}">
+        <gazebo>
+            <plugin name='gz::sim::systems::DiffDrive' filename='gz-sim-diff-drive-system'>
+                <!-- WHEEL INFORMATION -->
+                <left_joint>left_wheel_joint</left_joint>
+                <right_joint>right_wheel_joint</right_joint>
+                <wheel_separation>0.35</wheel_separation>
+                <wheel_radius>0.05</wheel_radius>
+                <!-- LIMITS -->
+                <!-- <max_wheel_torque>200</max_wheel_torque> -->
+                <!-- <max_wheel_acceleration>10.0</max_wheel_acceleration> -->
+                <!-- INPUT -->
+                <topic>cmd_vel</topic>
+                <!-- OUTPUT -->
+                <frame_id>odom</frame_id>
+                <child_frame_id>base_link</child_frame_id>
+                <odom_topic>odom</odom_topic>
+                <tf_topic>/tf</tf_topic>
+                <!-- <odom_publisher_frequency>30</odom_publisher_frequency> -->
+            </plugin>
+            <plugin name="gz::sim::systems::JointStatePublisher"
+                filename="gz-sim-joint-state-publisher-system">
+                <topic>joint_states</topic>
+                <joint_name>left_wheel_joint</joint_name>
+                <joint_name>right_wheel_joint</joint_name>
+            </plugin>
+        </gazebo>
+    </xacro:unless>
 </robot>

File: description/robot.urdf.xacro (robot description, xacro)
@@ -1,11 +1,19 @@
 <?xml version="1.0"?>
 <robot xmlns:xacro="http://www.ros.org/wiki/xacro"  name="robot">
+    <xacro:arg name="use_ros2_control" default="true" />
+    <xacro:arg name="use_sensor_fusion" default="true" />
+    <xacro:property name="use_ros2_control" value="$(arg use_ros2_control)" />
+    <xacro:property name="use_sensor_fusion" value="$(arg use_sensor_fusion)" />
     <xacro:include filename="robot_core.xacro" />
     <xacro:include filename="gazebo_control.xacro"/>
+    <xacro:include filename="ros2_control.xacro" />
     <xacro:include filename="lidar.xacro"/>
     <xacro:include filename="rgb_camera.xacro"/>
+    <xacro:include filename="depth_camera.xacro"/>
     <xacro:include filename="imu_sensor.xacro" />
-    <!-- <xacro:include filename="depth_camera.xacro"/> -->
-    <!-- <xacro:include filename="ros2_control.xacro" /> -->
-    <!-- <xacro:add_ros2_control left_joint="left_wheel_joint" right_joint="right_wheel_joint"/> -->
+    <xacro:add_ros2_control
+      left_joint="left_wheel_joint"
+      right_joint="right_wheel_joint"
+      use_ros2_control="${use_ros2_control}"
+      use_sensor_fusion="${use_sensor_fusion}" />
 </robot>
